Commit message: Updated urdf mass/inertai parameters, fixed axes confusion for wheels

File: src/eternal_bot_description/urdf/eternal_bot.xacro (robot description, xacro)
@@ -7,6 +7,6 @@
   <inertial>
     <origin xyz="0.0 0.0 0.025600000000000005" rpy="0 0 0"/>
-    <mass value="65.27180800000002"/>
-    <inertia ixx="0.440701" iyy="1.844045" izz="2.256229" ixy="0.0" iyz="0.0" ixz="0.0"/>
+    <mass value="14"/>
+    <inertia ixx="0.094525" iyy="0.395525" izz="0.483933" ixy="0.0" iyz="0.0" ixz="0.0"/>
   </inertial>
   <visual>
@@ -27,6 +27,6 @@
   <inertial>
     <origin xyz="-2.220446049250313e-16 0.025000000000000022 1.97758476261356e-16" rpy="0 0 0"/>
-    <mass value="3.0826877913349833"/>
-    <inertia ixx="0.002569" iyy="0.003853" izz="0.002569" ixy="0.0" iyz="0.0" ixz="0.0"/>
+    <mass value="0.4"/>
+    <inertia ixx="0.000333" iyy="0.0005" izz="0.000333" ixy="0.0" iyz="0.0" ixz="0.0"/>
   </inertial>
   <visual>
@@ -47,6 +47,6 @@
   <inertial>
     <origin xyz="2.220446049250313e-16 -0.025000000000000022 9.367506770274758e-17" rpy="0 0 0"/>
-    <mass value="3.0826877913349833"/>
-    <inertia ixx="0.002569" iyy="0.003853" izz="0.002569" ixy="0.0" iyz="-0.0" ixz="-0.0"/>
+    <mass value="0.4"/>
+    <inertia ixx="0.000333" iyy="0.0005" izz="0.000333" ixy="0.0" iyz="-0.0" ixz="-0.0"/>
   </inertial>
   <visual>
@@ -67,6 +67,6 @@
   <inertial>
     <origin xyz="-7.494005416219807e-16 -0.025000000000000022 -3.122502256758253e-17" rpy="0 0 0"/>
-    <mass value="3.0826877913349833"/>
-    <inertia ixx="0.002569" iyy="0.003853" izz="0.002569" ixy="-0.0" iyz="-0.0" ixz="-0.0"/>
+    <mass value="0.4"/>
+    <inertia ixx="0.000333" iyy="0.0005" izz="0.000333" ixy="-0.0" iyz="-0.0" ixz="-0.0"/>
   </inertial>
   <visual>
@@ -87,6 +87,6 @@
   <inertial>
     <origin xyz="0.0 0.025000000000000022 1.3773704399255848e-15" rpy="0 0 0"/>
-    <mass value="3.0826877913349833"/>
-    <inertia ixx="0.002569" iyy="0.003853" izz="0.002569" ixy="0.0" iyz="0.0" ixz="-0.0"/>
+    <mass value="0.4"/>
+    <inertia ixx="0.000333" iyy="0.0005" izz="0.000333" ixy="0.0" iyz="0.0" ixz="-0.0"/>
   </inertial>
   <visual>
@@ -107,6 +107,6 @@
   <inertial>
     <origin xyz="-5.790023100122029e-18 5.790023100122029e-18 0.025" rpy="0 0 0"/>
-    <mass value="3.082687791334984"/>
-    <inertia ixx="0.002569" iyy="0.002569" izz="0.003853" ixy="-0.0" iyz="-0.0" ixz="-0.0"/>
+    <mass value="0.15"/>
+    <inertia ixx="0.000125" iyy="0.000125" izz="0.0001875" ixy="-0.0" iyz="-0.0" ixz="-0.0"/>
   </inertial>
   <visual>
@@ -130,9 +130,9 @@
   <axis xyz="0.0 1.0 0.0"/>
 </joint>
-<joint name="front _right_joint" type="continuous">
+<joint name="front_right_joint" type="continuous">
   <origin xyz="0.22 -0.14 0.0256" rpy="0 0 0"/>
   <parent link="base_link"/>
   <child link="front_right_1"/>
-  <axis xyz="0.0 -1.0 0.0"/>
+  <axis xyz="0.0 1.0 0.0"/>
 </joint>
 <joint name="rear_right_joint" type="continuous">
@@ -140,5 +140,5 @@
   <parent link="base_link"/>
   <child link="rear_right_1"/>
-  <axis xyz="0.0 -1.0 0.0"/>
+  <axis xyz="0.0 1.0 0.0"/>
 </joint>
 <joint name="rear_left_joint" type="continuous">
