Commit message: Fix Gazebo skid-steer rotation and add documentation/learnings.md
- Wheel collisions: STL meshes -> cylinder primitives (mesh contacts ignored wheel friction)
- Anisotropic wheel friction (fdir1 along axle, mu1 0.3 lateral / mu2 1.0 rolling) so the
  long-wheelbase skid-steer can yaw; remove self_collide
- diff_drive_controller: wheel_separation 0.28 -> 0.33, drop dead use_stamped_vel, set frames/timeout
- Add twist_to_stamped relay (/cmd_vel Twist -> DDC TwistStamped), started in gazebo.launch.py
- Fix setup.cfg script dir (fusion2urdf_ros2 leftover), use_sim_time on robot_state_publisher
- documentation/learnings.md: root causes, physics explanations, workflow suggestions

Co-Authored-By: Claude Opus 5.5 <noreply@anthropic.com>

File: src/eternal_bot_description/urdf/eternal_bot.xacro (robot description, xacro)
@@ -37,8 +37,8 @@
     <material name="silver"/>
   </visual>
-  <collision>
-    <origin xyz="-0.22 -0.14 -0.0256" rpy="0 0 0"/>
+  <collision> <!-- cylinder, not STL: mesh contacts ignore surface friction in gz -->
+    <origin xyz="0 0.025 0" rpy="1.5708 0 0"/>
     <geometry>
-      <mesh filename="file://$(find eternal_bot_description)/meshes/front_left_1.stl" scale="0.001 0.001 0.001"/>
+      <cylinder radius="0.05" length="0.05"/>
     </geometry>
   </collision>
@@ -57,8 +57,8 @@
     <material name="silver"/>
   </visual>
-  <collision>
-    <origin xyz="-0.22 0.14 -0.0256" rpy="0 0 0"/>
+  <collision> <!-- cylinder, not STL: mesh contacts ignore surface friction in gz -->
+    <origin xyz="0 -0.025 0" rpy="1.5708 0 0"/>
     <geometry>
-      <mesh filename="file://$(find eternal_bot_description)/meshes/front_right_1.stl" scale="0.001 0.001 0.001"/>
+      <cylinder radius="0.05" length="0.05"/>
     </geometry>
   </collision>
@@ -77,8 +77,8 @@
     <material name="silver"/>
   </visual>
-  <collision>
-    <origin xyz="0.22 0.14 -0.0256" rpy="0 0 0"/>
+  <collision> <!-- cylinder, not STL: mesh contacts ignore surface friction in gz -->
+    <origin xyz="0 -0.025 0" rpy="1.5708 0 0"/>
     <geometry>
-      <mesh filename="file://$(find eternal_bot_description)/meshes/rear_right_1.stl" scale="0.001 0.001 0.001"/>
+      <cylinder radius="0.05" length="0.05"/>
     </geometry>
   </collision>
@@ -97,8 +97,8 @@
     <material name="silver"/>
   </visual>
-  <collision>
-    <origin xyz="0.22 -0.14 -0.0256" rpy="0 0 0"/>
+  <collision> <!-- cylinder, not STL: mesh contacts ignore surface friction in gz -->
+    <origin xyz="0 0.025 0" rpy="1.5708 0 0"/>
     <geometry>
-      <mesh filename="file://$(find eternal_bot_description)/meshes/rear_left_1.stl" scale="0.001 0.001 0.001"/>
+      <cylinder radius="0.05" length="0.05"/>
     </geometry>
   </collision>

Commit message: Simulate bot as holonomic using gz mecanum drive plugin
Replace gz_ros2_control/diff_drive with gz-sim-mecanum-drive-system, emulate
rollers via anisotropic wheel friction (sphere collisions, fdir1 pinned to
base_link at launch), bridge cmd_vel/odom/tf/joint_states.

Co-Authored-By: Claude Sonnet 5.5 <noreply@anthropic.com>

File: src/eternal_bot_description/urdf/eternal_bot.xacro (robot description, xacro)
@@ -2,5 +2,4 @@
 <robot name="eternal_bot" xmlns:xacro="http://www.ros.org/wiki/xacro">
 <xacro:include filename="$(find eternal_bot_description)/urdf/materials.xacro" />
-<xacro:include filename="$(find eternal_bot_description)/urdf/eternal_bot.ros2control" />
 <xacro:include filename="$(find eternal_bot_description)/urdf/eternal_bot.gazebo" />
 <link name="base_link">
@@ -37,8 +36,8 @@
     <material name="silver"/>
   </visual>
-  <collision> <!-- cylinder, not STL: mesh contacts ignore surface friction in gz -->
-    <origin xyz="0 0.025 0" rpy="1.5708 0 0"/>
+  <collision> <!-- sphere, not STL: mesh contacts ignore surface friction in gz; sphere + unrotated frame keeps fdir1 in link axes -->
+    <origin xyz="0 0.025 0" rpy="0 0 0"/>
     <geometry>
-      <cylinder radius="0.05" length="0.05"/>
+      <sphere radius="0.05"/>
     </geometry>
   </collision>
@@ -57,8 +56,8 @@
     <material name="silver"/>
   </visual>
-  <collision> <!-- cylinder, not STL: mesh contacts ignore surface friction in gz -->
-    <origin xyz="0 -0.025 0" rpy="1.5708 0 0"/>
+  <collision> <!-- sphere, not STL: mesh contacts ignore surface friction in gz; sphere + unrotated frame keeps fdir1 in link axes -->
+    <origin xyz="0 -0.025 0" rpy="0 0 0"/>
     <geometry>
-      <cylinder radius="0.05" length="0.05"/>
+      <sphere radius="0.05"/>
     </geometry>
   </collision>
@@ -77,8 +76,8 @@
     <material name="silver"/>
   </visual>
-  <collision> <!-- cylinder, not STL: mesh contacts ignore surface friction in gz -->
-    <origin xyz="0 -0.025 0" rpy="1.5708 0 0"/>
+  <collision> <!-- sphere, not STL: mesh contacts ignore surface friction in gz; sphere + unrotated frame keeps fdir1 in link axes -->
+    <origin xyz="0 -0.025 0" rpy="0 0 0"/>
     <geometry>
-      <cylinder radius="0.05" length="0.05"/>
+      <sphere radius="0.05"/>
     </geometry>
   </collision>
@@ -97,8 +96,8 @@
     <material name="silver"/>
   </visual>
-  <collision> <!-- cylinder, not STL: mesh contacts ignore surface friction in gz -->
-    <origin xyz="0 0.025 0" rpy="1.5708 0 0"/>
+  <collision> <!-- sphere, not STL: mesh contacts ignore surface friction in gz; sphere + unrotated frame keeps fdir1 in link axes -->
+    <origin xyz="0 0.025 0" rpy="0 0 0"/>
     <geometry>
-      <cylinder radius="0.05" length="0.05"/>
+      <sphere radius="0.05"/>
     </geometry>
   </collision>

Commit message: Add 2D gpu_lidar on lidar_1 and bridge /scan
Sensors system loaded from the model; lidar_1 raised to z=0.1062 (top of
the mesh) so the scan plane clears the wheel tops. /scan bridged GZ->ROS.
Drive test passes on all 10 cases.

Co-Authored-By: Claude Sonnet 5.5 <noreply@anthropic.com>

File: src/eternal_bot_description/urdf/eternal_bot.xacro (robot description, xacro)
@@ -105,10 +105,10 @@
 <link name="lidar_1">
   <inertial>
-    <origin xyz="-5.790023100122029e-18 5.790023100122029e-18 0.025" rpy="0 0 0"/>
+    <origin xyz="-5.790023100122029e-18 5.790023100122029e-18 -0.03" rpy="0 0 0"/>
     <mass value="0.15"/>
     <inertia ixx="0.000125" iyy="0.000125" izz="0.0001875" ixy="-0.0" iyz="-0.0" ixz="-0.0"/>
   </inertial>
   <visual>
-    <origin xyz="-0.0 -0.0 -0.0512" rpy="0 0 0"/>
+    <origin xyz="-0.0 -0.0 -0.1062" rpy="0 0 0"/>
     <geometry>
       <mesh filename="file://$(find eternal_bot_description)/meshes/lidar_1.stl" scale="0.001 0.001 0.001"/>
@@ -117,5 +117,5 @@
   </visual>
   <collision>
-    <origin xyz="-0.0 -0.0 -0.0512" rpy="0 0 0"/>
+    <origin xyz="-0.0 -0.0 -0.1062" rpy="0 0 0"/>
     <geometry>
       <mesh filename="file://$(find eternal_bot_description)/meshes/lidar_1.stl" scale="0.001 0.001 0.001"/>
@@ -148,5 +148,5 @@
 </joint>
 <joint name="lidar_joint" type="fixed">
-  <origin xyz="0.0 0.0 0.0512" rpy="0 0 0"/>
+  <origin xyz="0.0 0.0 0.1062" rpy="0 0 0"/>
   <parent link="base_link"/>
   <child link="lidar_1"/>
